Commit message: add imu and hall sensor to robot urdf

File: src/robot_urdf/urdf/properties.xacro (robot description, xacro)
@@ -12,3 +12,6 @@
         <color rgba="0.0 0.0 0.0 1.0" />
     </material>
+    <material name="colors_blue">
+        <color rgba="0.56 0.82 1.0 1.0" />
+    </material>
 </robot>

File: src/robot_urdf/urdf/robot.urdf.xacro (robot description, xacro)
@@ -35,3 +35,10 @@
     <xacro:ultrasound_sensor name="ultrasound_2" rpy="-0.698 1.5708 0" xyz="0.1494 0.1254 0" />
     <xacro:ultrasound_sensor name="ultrasound_3" rpy="0.698 1.5708 0" xyz="0.1494 -0.1254 0" />
+    <!-- ===> IMU <=== -->
+    <xacro:include filename="imu.xacro" />
+    <xacro:imu />
+    <!-- ===> HALL SENSOR <=== -->
+    <xacro:include filename="hall_sensor.xacro" />
+    <xacro:hall_sensor name="left" x="-0.0235" y="0.0125" rotate="0.0" />
+    <xacro:hall_sensor name="right" x="0.0235" y="-0.0125" rotate="3.1411" />
 </robot>

File: src/robot_urdf/urdf/robot_base.xacro (robot description, xacro)
@@ -8,5 +8,7 @@
                     <cylinder radius="0.2" length="${robot_base_hight}" />
                 </geometry>
-                <material name="colors_gray" />
+                <material name="colors_grayd">
+                    <color rgba="0.66 0.66 0.66 0.75" />
+                </material>
             </visual>
         </link>
