Commit message: update lidar launch file

File: src/robot_urdf/urdf/robot_base.xacro (robot description, xacro)
@@ -8,7 +8,5 @@
                     <cylinder radius="0.2" length="${robot_base_hight}" />
                 </geometry>
-                <material name="colors_grayd">
-                    <color rgba="0.66 0.66 0.66 0.75" />
-                </material>
+                <material name="colors_gray"/>
             </visual>
         </link>

File: src/robot_urdf/urdf/wheel.xacro (robot description, xacro)
@@ -25,5 +25,5 @@
         </link>
         <!-- Joint-->
-        <joint name="${name}_joint" type="continuous">
+        <joint name="${name}_joint" type="fixed">
             <parent link="robot_base_link" />
             <child link="${name}" />
